Commit message: add: use xacro variables/properties

File: ros2_workspace/src/my_robot_description/urdf/my_robot.urdf.xacro (robot description, xacro)
@@ -1,4 +1,5 @@
 <?xml version="1.0"?>
 <robot name = "my_robot" xmlns:xacro="http://www.ros.org/wiki/xacro">
+    <xacro:property name = "base_length" value = "0.6"/>
     <material name = "blue">
         <color rgba = "0 0 0.7 1"/>
@@ -10,5 +11,5 @@
         <visual>
             <geometry>
-                <box size = "0.6 0.4 0.2"/>
+                <box size = "${base_length} 0.4 0.2"/>
             </geometry>
             <!--z=0.1, which is half of height of box size, it keeps box on the origin.-->
@@ -22,5 +23,5 @@
                 <cylinder radius="0.1" length="0.05" />
             </geometry>
-            <origin xyz = "0 0 0" rpy = "1.57 0 0"/>
+            <origin xyz = "0 0 0" rpy = "${pi/2.0} 0 0"/>
             <material name = "grey"/>
         </visual>
@@ -31,5 +32,5 @@
                 <cylinder radius="0.1" length="0.05" />
             </geometry>
-            <origin xyz = "0 0 0" rpy = "1.57 0 0"/>
+            <origin xyz = "0 0 0" rpy = "${pi/2.0} 0 0"/>
             <material name = "grey"/>
         </visual>
@@ -40,5 +41,5 @@
                 <sphere radius = "0.05" />
             </geometry>
-            <origin xyz = "0 0 0" rpy = "1.57 0 0"/>
+            <origin xyz = "0 0 0" rpy = "0 0 0"/>
             <material name = "grey"/>
         </visual>
@@ -48,5 +49,5 @@
         <parent link = "base_link"/>
         <child link = "right_wheel_link"/>
-        <origin xyz = "-0.15 -0.225 0"  rpy = "0 0 0"/>
+        <origin xyz = "${-base_length/4.0} -0.225 0"  rpy = "0 0 0"/>
         <axis xyz = "0 1 0"/>
     </joint>
@@ -54,5 +55,5 @@
         <parent link = "base_link"/>
         <child link = "left_wheel_link"/>
-        <origin xyz = "-0.15 0.225 0"  rpy = "0 0 0"/>
+        <origin xyz = "${-base_length/4.0} 0.225 0"  rpy = "0 0 0"/>
         <axis xyz = "0 1 0"/>
     </joint>
@@ -60,5 +61,5 @@
         <parent link = "base_link"/>
         <child link = "caster_wheel_link"/>
-        <origin xyz = "0.2 0 -0.05"  rpy = "0 0 0"/>
+        <origin xyz = "${base_length/3.0} 0 -0.05"  rpy = "0 0 0"/>
     </joint>
     <joint name = "base_joint" type = "fixed">

Commit message: modify: change hard-coded values to xacro variables

File: ros2_workspace/src/my_robot_description/urdf/my_robot.urdf.xacro (robot description, xacro)
@@ -2,4 +2,9 @@
 <robot name = "my_robot" xmlns:xacro="http://www.ros.org/wiki/xacro">
     <xacro:property name = "base_length" value = "0.6"/>
+    <xacro:property name = "base_width" value = "0.4"/>
+    <xacro:property name = "base_height" value = "0.2"/>
+    <xacro:property name = "wheel_radius" value = "0.1"/>
+    <xacro:property name = "wheel_length" value = "0.05"/>
+    <xacro:property name = "caster_wheel_radius" value = "0.05"/>
     <material name = "blue">
         <color rgba = "0 0 0.7 1"/>
@@ -11,8 +16,8 @@
         <visual>
             <geometry>
-                <box size = "${base_length} 0.4 0.2"/>
+                <box size = "${base_length} ${base_width} ${base_height}"/>
             </geometry>
             <!--z=0.1, which is half of height of box size, it keeps box on the origin.-->
-            <origin xyz = "0 0 0.1" rpy = "0 0 0"/>
+            <origin xyz = "0 0 ${base_height/2.0}" rpy = "0 0 0"/>
             <material name = "blue"/>
         </visual>
@@ -21,5 +26,5 @@
         <visual>
             <geometry>
-                <cylinder radius="0.1" length="0.05" />
+                <cylinder radius="${wheel_radius}" length="${wheel_length}" />
             </geometry>
             <origin xyz = "0 0 0" rpy = "${pi/2.0} 0 0"/>
@@ -30,5 +35,5 @@
         <visual>
             <geometry>
-                <cylinder radius="0.1" length="0.05" />
+                <cylinder radius="${wheel_radius}" length="${wheel_length}" />
             </geometry>
             <origin xyz = "0 0 0" rpy = "${pi/2.0} 0 0"/>
@@ -39,5 +44,5 @@
         <visual>
             <geometry>
-                <sphere radius = "0.05" />
+                <sphere radius = "${caster_wheel_radius}" />
             </geometry>
             <origin xyz = "0 0 0" rpy = "0 0 0"/>
@@ -49,5 +54,5 @@
         <parent link = "base_link"/>
         <child link = "right_wheel_link"/>
-        <origin xyz = "${-base_length/4.0} -0.225 0"  rpy = "0 0 0"/>
+        <origin xyz = "${-base_length/4.0} ${-base_width/2.0 + (-wheel_length/2.0)} 0"  rpy = "0 0 0"/>
         <axis xyz = "0 1 0"/>
     </joint>
@@ -55,5 +60,5 @@
         <parent link = "base_link"/>
         <child link = "left_wheel_link"/>
-        <origin xyz = "${-base_length/4.0} 0.225 0"  rpy = "0 0 0"/>
+        <origin xyz = "${-base_length/4.0} ${base_width/2.0 + wheel_length/2.0} 0"  rpy = "0 0 0"/>
         <axis xyz = "0 1 0"/>
     </joint>
@@ -61,10 +66,10 @@
         <parent link = "base_link"/>
         <child link = "caster_wheel_link"/>
-        <origin xyz = "${base_length/3.0} 0 -0.05"  rpy = "0 0 0"/>
+        <origin xyz = "${base_length/3.0} 0 ${-caster_wheel_radius}"  rpy = "0 0 0"/>
     </joint>
     <joint name = "base_joint" type = "fixed">
         <parent link = "base_footprint_link"/>
         <child link = "base_link"/>
-        <origin xyz = "0 0 0.1"  rpy = "0 0 0"/>
+        <origin xyz = "0 0 ${wheel_radius}"  rpy = "0 0 0"/>
     </joint>
 </robot>

Commit message: modify: change caster_wheel_radius to wheel_radius/2.0

File: ros2_workspace/src/my_robot_description/urdf/my_robot.urdf.xacro (robot description, xacro)
@@ -3,8 +3,7 @@
     <xacro:property name = "base_length" value = "0.6"/>
     <xacro:property name = "base_width" value = "0.4"/>
-    <xacro:property name = "base_height" value = "0.2"/>
-    <xacro:property name = "wheel_radius" value = "0.1"/>
-    <xacro:property name = "wheel_length" value = "0.05"/>
-    <xacro:property name = "caster_wheel_radius" value = "0.05"/>
+    <xacro:property name = "base_height" value = "0.1"/>
+    <xacro:property name = "wheel_radius" value = "0.05"/>
+    <xacro:property name = "wheel_length" value = "0.1"/>
     <material name = "blue">
         <color rgba = "0 0 0.7 1"/>
@@ -44,5 +43,5 @@
         <visual>
             <geometry>
-                <sphere radius = "${caster_wheel_radius}" />
+                <sphere radius = "${wheel_radius/2.0}" />
             </geometry>
             <origin xyz = "0 0 0" rpy = "0 0 0"/>
@@ -66,5 +65,5 @@
         <parent link = "base_link"/>
         <child link = "caster_wheel_link"/>
-        <origin xyz = "${base_length/3.0} 0 ${-caster_wheel_radius}"  rpy = "0 0 0"/>
+        <origin xyz = "${base_length/3.0} 0 ${-wheel_radius/2.0}"  rpy = "0 0 0"/>
     </joint>
     <joint name = "base_joint" type = "fixed">

Commit message: modify: set caster_wheel_radius to half of wheel_radius

File: ros2_workspace/src/my_robot_description/urdf/my_robot.urdf.xacro (robot description, xacro)
@@ -44,5 +44,5 @@
         <visual>
             <geometry>
-                <sphere radius = "${caster_wheel_radius}" />
+                <sphere radius = "${wheel_radius/2.0}" />
             </geometry>
             <origin xyz = "0 0 0" rpy = "0 0 0"/>
@@ -66,5 +66,5 @@
         <parent link = "base_link"/>
         <child link = "caster_wheel_link"/>
-        <origin xyz = "${base_length/3.0} 0 ${-caster_wheel_radius}"  rpy = "0 0 0"/>
+        <origin xyz = "${base_length/3.0} 0 ${-wheel_radius/2.0}"  rpy = "0 0 0"/>
     </joint>
     <joint name = "base_joint" type = "fixed">

Commit message: modify: set caster wheel radius to half of wheel radius

File: ros2_workspace/src/my_robot_description/urdf/my_robot.urdf.xacro (robot description, xacro)
@@ -3,7 +3,7 @@
     <xacro:property name = "base_length" value = "0.6"/>
     <xacro:property name = "base_width" value = "0.4"/>
-    <xacro:property name = "base_height" value = "0.1"/>
-    <xacro:property name = "wheel_radius" value = "0.05"/>
-    <xacro:property name = "wheel_length" value = "0.1"/>
+    <xacro:property name = "base_height" value = "0.2"/>
+    <xacro:property name = "wheel_radius" value = "0.1"/>
+    <xacro:property name = "wheel_length" value = "0.05"/>
     <material name = "blue">
         <color rgba = "0 0 0.7 1"/>
